File: kicad/version_1/working/working.kicad_pcb (KiCad board)
At the start: 2 copper layers, 13 x 33 mm, 6 parts

Commit message: version 2
Parts:
- removed the CONN2 at (-2.54, -17.8)
- CONN1: value hi13pth_electronic_header_2_54_mm_3_pin_through_hole -> hi16pth_electronic_header_2_54_mm_6_pin_through_hole; footprint oomlout_oomp_part_footprints:hi13pth_electronic_header_2_54_mm_3_pin_through_hole -> oomlout_oomp_part_footprints:hi16pth_electronic_header_2_54_mm_6_pin_through_hole
- moved CONN1 3.81 mm to (-6.35, -15.2)
- renumbered CONN3 to CONN2, CONN4 to CONN3
Routing:
- net enc: track 26.5 -> 24.4 mm
- net switch_a: track 26.5 -> 24.4 mm
- net gnd: track 28.9 -> 27.0 mm
- net b: track 27.6 -> 29.2 mm
- net 5v: track 27.6 -> 29.2 mm
- net a: track 27.8 -> 29.2 mm
Other:
- board size 13 x 33 mm -> 16 x 32 mm
- board text removed: "a b 5v"
- board text removed: "enc wd gnd sb"
