File: kicad/version_1/working/working.kicad_sch (KiCad schematic)
At the start: 4 parts

Commit message: version 2
Parts:
- removed CONN1, CONN2: hi13pth_electronic_header_2_54_mm_3_pin_through_h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, oomlout_oomp_part_footprints:hi13pth_electronic_header_2_54_mm_3_pin_through_hole, symbol oomp:hi13pth_electronic_header_2_54_mm_3_pin_through_hole
- added CONN1: hi16pth_electronic_header_2_54_mm_6_pin_through_h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, oomlout_oomp_part_footprints:hi16pth_electronic_header_2_54_mm_6_pin_through_hole, symbol oomp:hi16pth_electronic_header_2_54_mm_6_pin_through_hole
- renumbered CONN3 to CONN2, CONN4 to CONN3
Connections:
- net 5v: now also CONN1.3 (Pin_3)
- net a: now also CONN1.1 (Pin_1)
- net b: now also CONN1.2 (Pin_2)
- net enc: now also CONN1.4 (Pin_4)
- net gnd: now also CONN1.6 (Pin_6)
- net switch_a: now also CONN1.5 (Pin_5)
Changed lines of the file:
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@@
     )
   )
-  (symbol (lib_id "oomp:hi13pth_electronic_header_2_54_mm_3_pin_through_hole") (at 40.64 54.61 0) (unit 1)
-    (in_bom yes) (on_board yes) (dnp no)
-    (property "Reference" "CONN2" (at 34.29 53.34 0)
-      (effects (font (size 1.27 1.27)) (justify right))
+  (symbol (lib_id "oomp:hi16pth_electronic_header_2_54_mm_6_pin_through_hole") (at 40.64 49.53 0) (unit 1)
+    (in_bom yes) (on_board yes) (dnp no) (fields_autoplaced)
+    (property "Reference" "CONN1" (at 41.275 39.37 0)
+      (effects (font (size 1.27 1.27)))
     )
-    (property "Value" "hi13pth_electronic_header_2_54_mm_3_pin_through_hole" (at 34.29 55.88 0)
-      (effects (font (size 1.27 1.27)) (justify right))
+    (property "Value" "hi16pth_electronic_header_2_54_mm_6_pin_through_hole" (at 41.275 41.91 0)
+      (effects (font (size 1.27 1.27)))
     )
-    (property "Footprint" "oomlout_oomp_part_footprints:hi13pth_electronic_header_2_54_mm_3_pin_through_hole" (at 40.64 54.61 0)
+    (property "Footprint" "oomlout_oomp_part_footprints:hi16pth_electronic_header_2_54_mm_6_pin_through_hole" (at 40.64 49.53 0)
       (effects (font (size 1.27 1.27)) hide)
     )
-    (property "Datasheet" "https://github.com/oomlout/oomlout_oomp_v3/parts/electronic_header_2_54_mm_3_pin_through_hole/datasheet.pdf" (at 40.64 54.61 0)
+    (property "Datasheet" "https://github.com/oomlout/oomlout_oomp_v3/parts/electronic_header_2_54_mm_6_pin_through_hole/datasheet.pdf" (at 40.64 49.53 0)
       (effects (font (size 1.27 1.27)) hide)
     )
@@
     (pin "2")
     (pin "3")
+    (pin "4")
+    (pin "5")
+    (pin "6")
     (instances
       (project "working"
         (path "/c9993764-076f-44f6-bf4c-6b69ce17c9e4"
-          (reference "CONN2") (unit 1)
+          (reference "CONN1") (unit 1)
         )
       )
@@
   (symbol (lib_id "oomp:hi13pth_electronic_header_2_54_mm_3_pin_through_hole") (at 100.33 46.99 0) (mirror y) (unit 1)
     (in_bom yes) (on_board yes) (dnp no)
-    (property "Reference" "CONN3" (at 106.68 45.72 0)
+    (property "Reference" "CONN2" (at 106.68 45.72 0)
       (effects (font (size 1.27 1.27)) (justify right))
     )
@@
       (project "working"
         (path "/c9993764-076f-44f6-bf4c-6b69ce17c9e4"
-          (reference "CONN3") (unit 1)
-        )
-      )
-    )
-  )
-  (symbol (lib_id "oomp:hi13pth_electronic_header_2_54_mm_3_pin_through_hole") (at 40.64 46.99 0) (unit 1)
-    (in_bom yes) (on_board yes) (dnp no)
-    (property "Reference" "CONN1" (at 34.29 45.72 0)
-      (effects (font (size 1.27 1.27)) (justify right))
-    )
-    (property "Value" "hi13pth_electronic_header_2_54_mm_3_pin_through_hole" (at 34.29 48.26 0)
-      (effects (font (size 1.27 1.27)) (justify right))
-    )
-    (property "Footprint" "oomlout_oomp_part_footprints:hi13pth_electronic_header_2_54_mm_3_pin_through_hole" (at 40.64 46.99 0)
-      (effects (font (size 1.27 1.27)) hide)
-    )
-    (property "Datasheet" "https://github.com/oomlout/oomlout_oomp_v3/parts/electronic_header_2_54_mm_3_pin_through_hole/datasheet.pdf" (at 40.64 46.99 0)
-      (effects (font (size 1.27 1.27)) hide)
-    )
-    (pin "1")
-    (pin "2")
-    (pin "3")
-    (instances
-      (project "working"
-        (path "/c9993764-076f-44f6-bf4c-6b69ce17c9e4"
-          (reference "CONN1") (unit 1)
+          (reference "CONN2") (unit 1)
         )
       )
@@
   (symbol (lib_id "oomp:hi14pth_electronic_header_2_54_mm_4_pin_through_hole") (at 100.33 54.61 0) (mirror y) (unit 1)
     (in_bom yes) (on_board yes) (dnp no)
-    (property "Reference" "CONN4" (at 106.68 54.61 0)
+    (property "Reference" "CONN3" (at 106.68 54.61 0)
       (effects (font (size 1.27 1.27)) (justify right))
     )
@@
       (project "working"
         (path "/c9993764-076f-44f6-bf4c-6b69ce17c9e4"
-          (reference "CONN4") (unit 1)
+          (reference "CONN3") (unit 1)
         )
       )
